File: cad/se7en.sch (EAGLE design)
At the start: 67 parts, among them CN1 MICROSD-EJECT, CN3 DO NOT PLACE, CN4 DO NOT PLACE, CN5 DO NOT PLACE, CN6 DO NOT PLACE, CN7 DO NOT PLACE, Q1 FDC6329S, SW1 SWITCHKMR211, SW2 SWITCHKMR211, U1 ATSAME70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

Commit message: tweak
Parts:
- U1: value ATSAME70 -> ATSAMS70
- renumbered LOGO1 to LOGO$1
Changed lines of the file:
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@@
 <parts>
 <part name="FRAME1" library="frames" deviceset="FRAME_B_L" device=""/>
-<part name="U1" library="jaw" deviceset="ATSAME70" device=""/>
+<part name="U1" library="jaw" deviceset="ATSAME70" device="" value="ATSAMS70"/>
 <part name="GND1" library="jaw" deviceset="PWR-GND" device=""/>
 <part name="VCC1" library="jaw" deviceset="PWR-VCC" device=""/>
@@
 <part name="U$1" library="jaw" deviceset="ROBOTMAN-LOGO" device="2"/>
 <part name="U$3" library="jaw" deviceset="ROBOTMAN-LOGO" device="2"/>
-<part name="LOGO1" library="SparkFun-Aesthetics" deviceset="OSHW-LOGO" device="M"/>
+<part name="LOGO$1" library="SparkFun-Aesthetics" deviceset="OSHW-LOGO" device="M"/>
 <part name="U2" library="jaw" deviceset="MCP73831" device=""/>
 <part name="VR1" library="jaw" deviceset="REGULATOR4" device="-SOT23" value="3v3, 500mA"/>
@@
 <instance part="U$1" gate="G$1" x="332.74" y="25.4"/>
 <instance part="U$3" gate="G$1" x="342.9" y="25.4"/>
-<instance part="LOGO1" gate="G$1" x="414.02" y="27.94"/>
+<instance part="LOGO$1" gate="G$1" x="414.02" y="27.94"/>
 <instance part="U2" gate="G$1" x="43.18" y="55.88"/>
 <instance part="VR1" gate="G$1" x="60.96" y="20.32"/>

Commit message: fix typo
Parts:
- Q1: value FDC6329S -> FDC6392S; device jaw:FDC6329S -> jaw:FDC6392S
Changed lines of the file:
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@@
 <part name="R8" library="jaw" deviceset="R" device="-0402" value="1k"/>
 <part name="LED2" library="jaw" deviceset="LED-DUAL" device="0805"/>
-<part name="Q1" library="jaw" deviceset="FDC6329S" device=""/>
+<part name="Q1" library="jaw" deviceset="FDC6392S" device=""/>
 <part name="GND18" library="jaw" deviceset="PWR-GND" device=""/>
 <part name="R9" library="jaw" deviceset="R" device="-0402" value="10k"/>
