File: cad/se7en.sch (EAGLE design)
At the start: 67 parts, among them CN1 MICROSD-EJECT, CN3 DO NOT PLACE, CN4 DO NOT PLACE, CN5 DO NOT PLACE, CN6 DO NOT PLACE, CN7 DO NOT PLACE, Q1 FDC6392S, SW1 SWITCHKMR211, SW2 SWITCHKMR211, U1 ATSAMS70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

Commit message: remove pullups (use pio pullups)
Parts:
- removed R6: 100k, jaw:R-ARRAY40603-ARV
- added R12: 100k, jaw:R-0402
- C25: value 10u -> 10u 10V
- L4: value 10u -> 10uH
- R4: device jaw:R-ARRAY40603-ARV -> jaw:R-0402
Connections:
- net CARDIO: now also U1.PD16; no longer R6B.2
- net SDIOCM: no longer R6A.2
- net SDIOD0: no longer R4D.2
- net SDIOD1: no longer R4R.2
- net SDIOD2: no longer R4B.2
- net SDIOD3: no longer R4A.2
- net SWCLK: now also R12.P$1; no longer R6D.2
- net SWDIO: now also R4.P$1; no longer R6R.2
- net VCC: now also R12.P$2, R4.P$2; no longer R4A.1, R4B.1, R4D.1, R4R.1, R6A.1, R6B.1, R6D.1, R6R.1
Changed lines of the file:
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@@
 <part name="C2" library="jaw" deviceset="C" device="-0402" value=".1u"/>
 <part name="C3" library="jaw" deviceset="C" device="-0402" value=".1u"/>
-<part name="L4" library="jaw" deviceset="L" device="SMD0603" value="10u"/>
+<part name="L4" library="jaw" deviceset="L" device="SMD0603" value="10uH"/>
 <part name="R2" library="jaw" deviceset="R" device="-0402" value="5k62 1%"/>
 <part name="C4" library="jaw" deviceset="C" device="0603" value="10u"/>
@@
 <part name="R1" library="jaw" deviceset="R" device="-0402" value="10k"/>
 <part name="R3" library="jaw" deviceset="R" device="-0402" value="10k"/>
-<part name="R4" library="jaw" deviceset="R-ARRAY4" device="0603-ARV" value="100k"/>
 <part name="C24" library="jaw" deviceset="C" device="0603" value="4u7"/>
 <part name="F1" library="jaw" deviceset="FUSE" device="" value="750mA"/>
@@
 <part name="GND14" library="jaw" deviceset="PWR-GND" device=""/>
 <part name="GND15" library="jaw" deviceset="PWR-GND" device=""/>
-<part name="R6" library="jaw" deviceset="R-ARRAY4" device="0603-ARV" value="100k"/>
 <part name="GND16" library="jaw" deviceset="PWR-GND" device=""/>
-<part name="VCC8" library="jaw" deviceset="PWR-VCC" device=""/>
 <part name="VCC9" library="jaw" deviceset="PWR-VCC" device=""/>
 <part name="GND17" library="jaw" deviceset="PWR-GND" device=""/>
@@
 <part name="CN6" library="jaw" deviceset="HEADER-1X1" device="SMALL" value="DO NOT PLACE"/>
 <part name="CN7" library="jaw" deviceset="HEADER-1X1" device="SMALL" value="DO NOT PLACE"/>
-<part name="C25" library="jaw" deviceset="C" device="0603" value="10u"/>
+<part name="C25" library="jaw" deviceset="C" device="0603" value="10u 10V"/>
+<part name="R4" library="jaw" deviceset="R" device="-0402" value="100k"/>
+<part name="R12" library="jaw" deviceset="R" device="-0402" value="100k"/>
+<part name="VCC10" library="jaw" deviceset="PWR-VCC" device=""/>
 </parts>
 <sheets>
@@
 <instance part="R1" gate="G$1" x="71.12" y="251.46" rot="R90"/>
 <instance part="R3" gate="G$1" x="71.12" y="213.36" rot="R90"/>
-<instance part="R4" gate="A" x="342.9" y="124.46" rot="R180"/>
-<instance part="R4" gate="B" x="342.9" y="129.54" rot="R180"/>
-<instance part="R4" gate="R" x="342.9" y="134.62" rot="R180"/>
-<instance part="R4" gate="D" x="342.9" y="139.7" rot="R180"/>
 <instance part="C24" gate="G$1" x="363.22" y="142.24" rot="R180"/>
 <instance part="F1" gate="G$1" x="22.86" y="71.12"/>
@@
 <instance part="GND14" gate="G$1" x="45.72" y="236.22"/>
 <instance part="GND15" gate="G$1" x="71.12" y="205.74"/>
-<instance part="R6" gate="A" x="342.9" y="99.06" rot="R180"/>
-<instance part="R6" gate="B" x="342.9" y="104.14" rot="R180"/>
-<instance part="R6" gate="R" x="342.9" y="109.22" rot="R180"/>
-<instance part="R6" gate="D" x="342.9" y="114.3" rot="R180"/>
 <instance part="GND16" gate="G$1" x="408.94" y="101.6"/>
-<instance part="VCC8" gate="G$1" x="347.98" y="147.32"/>
 <instance part="VCC9" gate="G$1" x="363.22" y="147.32"/>
 <instance part="GND17" gate="G$1" x="363.22" y="132.08"/>
@@
 <instance part="CN7" gate="G$1" x="53.34" y="132.08" rot="R180"/>
 <instance part="C25" gate="G$1" x="40.64" y="15.24"/>
+<instance part="R4" gate="G$1" x="416.56" y="73.66" rot="R90"/>
+<instance part="R12" gate="G$1" x="421.64" y="73.66" rot="R90"/>
+<instance part="VCC10" gate="G$1" x="419.1" y="83.82"/>
 </instances>
 <busses>
@@
 </segment>
 <segment>
-<pinref part="R6" gate="A" pin="1"/>
-<pinref part="R6" gate="B" pin="1"/>
-<wire x1="347.98" y1="99.06" x2="347.98" y2="104.14" width="0.1524" layer="91"/>
-<pinref part="R6" gate="R" pin="1"/>
-<wire x1="347.98" y1="104.14" x2="347.98" y2="109.22" width="0.1524" layer="91"/>
-<junction x="347.98" y="104.14"/>
-<pinref part="R6" gate="D" pin="1"/>
-<wire x1="347.98" y1="109.22" x2="347.98" y2="114.3" width="0.1524" layer="91"/>
-<junction x="347.98" y="109.22"/>
-<pinref part="R4" gate="A" pin="1"/>
-<wire x1="347.98" y1="114.3" x2="347.98" y2="124.46" width="0.1524" layer="91"/>
-<junction x="347.98" y="114.3"/>
-<pinref part="R4" gate="B" pin="1"/>
-<wire x1="347.98" y1="124.46" x2="347.98" y2="129.54" width="0.1524" layer="91"/>
-<junction x="347.98" y="124.46"/>
-<pinref part="R4" gate="R" pin="1"/>
-<wire x1="347.98" y1="129.54" x2="347.98" y2="134.62" width="0.1524" layer="91"/>
-<junction x="347.98" y="129.54"/>
-<pinref part="R4" gate="D" pin="1"/>
-<wire x1="347.98" y1="134.62" x2="347.98" y2="139.7" width="0.1524" layer="91"/>
-<junction x="347.98" y="134.62"/>
-<wire x1="347.98" y1="139.7" x2="347.98" y2="144.78" width="0.1524" layer="91"/>
-<junction x="347.98" y="139.7"/>
-<pinref part="VCC8" gate="G$1" pin="VCC"/>
-</segment>
-<segment>
 <pinref part="C24" gate="G$1" pin="P$2"/>
 <pinref part="VCC9" gate="G$1" pin="VCC"/>
@@
 <wire x1="353.06" y1="175.26" x2="347.98" y2="175.26" width="0.1524" layer="91"/>
 <label x="340.36" y="175.26" size="1.27" layer="95"/>
+</segment>
+<segment>
+<pinref part="R4" gate="G$1" pin="P$2"/>
+<wire x1="416.56" y1="78.74" x2="416.56" y2="81.28" width="0.1524" layer="91"/>
+<pinref part="R12" gate="G$1" pin="P$2"/>
+<wire x1="416.56" y1="81.28" x2="419.1" y2="81.28" width="0.1524" layer="91"/>
+<wire x1="419.1" y1="81.28" x2="421.64" y2="81.28" width="0.1524" layer="91"/>
+<wire x1="421.64" y1="81.28" x2="421.64" y2="78.74" width="0.1524" layer="91"/>
+<pinref part="VCC10" gate="G$1" pin="VCC"/>
+<junction x="419.1" y="81.28"/>
 </segment>
 </net>
@@
 <wire x1="403.86" y1="63.5" x2="406.4" y2="63.5" width="0.1524" layer="91"/>
 <label x="406.4" y="63.5" size="1.27" layer="95"/>
-</segment>
-<segment>
-<pinref part="R6" gate="D" pin="2"/>
-<wire x1="337.82" y1="114.3" x2="335.28" y2="114.3" width="0.1524" layer="91"/>
-<label x="327.66" y="114.3" size="1.27" layer="95"/>
+<pinref part="R12" gate="G$1" pin="P$1"/>
+<wire x1="406.4" y1="63.5" x2="421.64" y2="63.5" width="0.1524" layer="91"/>
+<wire x1="421.64" y1="63.5" x2="421.64" y2="68.58" width="0.1524" layer="91"/>
 </segment>
 </net>
@@
 <wire x1="403.86" y1="66.04" x2="406.4" y2="66.04" width="0.1524" layer="91"/>
 <label x="406.4" y="66.04" size="1.27" layer="95"/>
-</segment>
-<segment>
-<pinref part="R6" gate="R" pin="2"/>
-<wire x1="337.82" y1="109.22" x2="335.28" y2="109.22" width="0.1524" layer="91"/>
-<label x="327.66" y="109.22" size="1.27" layer="95"/>
+<pinref part="R4" gate="G$1" pin="P$1"/>
+<wire x1="406.4" y1="66.04" x2="416.56" y2="66.04" width="0.1524" layer="91"/>
+<wire x1="416.56" y1="66.04" x2="416.56" y2="68.58" width="0.1524" layer="91"/>
 </segment>
 </net>
@@
 <label x="157.48" y="109.22" size="1.27" layer="95"/>
 </segment>
-<segment>
-<pinref part="R4" gate="D" pin="2"/>
-<wire x1="337.82" y1="139.7" x2="335.28" y2="139.7" width="0.1524" layer="91"/>
-<label x="327.66" y="139.7" size="1.27" layer="95"/>
-</segment>
 </net>
 <net name="SDIOD1" class="0">
@@
 <label x="157.48" y="106.68" size="1.27" layer="95"/>
 </segment>
-<segment>
-<pinref part="R4" gate="R" pin="2"/>
-<wire x1="337.82" y1="134.62" x2="335.28" y2="134.62" width="0.1524" layer="91"/>
-<label x="327.66" y="134.62" size="1.27" layer="95"/>
-</segment>
 </net>
 <net name="SDIOD2" class="0">
@@
 <label x="157.48" y="119.38" size="1.27" layer="95"/>
 </segment>
-<segment>
-<pinref part="R4" gate="B" pin="2"/>
-<wire x1="337.82" y1="129.54" x2="335.28" y2="129.54" width="0.1524" layer="91"/>
-<label x="327.66" y="129.54" size="1.27" layer="95"/>
-</segment>
 </net>
 <net name="SDIOD3" class="0">
@@
 <label x="157.48" y="116.84" size="1.27" layer="95"/>
 </segment>
-<segment>
-<pinref part="R4" gate="A" pin="2"/>
-<wire x1="337.82" y1="124.46" x2="335.28" y2="124.46" width="0.1524" layer="91"/>
-<label x="327.66" y="124.46" size="1.27" layer="95"/>
-</segment>
 </net>
 <net name="SDIOCK" class="0">
@@
 <label x="157.48" y="114.3" size="1.27" layer="95"/>
 </segment>
-<segment>
-<pinref part="R6" gate="A" pin="2"/>
-<wire x1="337.82" y1="99.06" x2="335.28" y2="99.06" width="0.1524" layer="91"/>
-<label x="327.66" y="99.06" size="1.27" layer="95"/>
-</segment>
 </net>
 <net name="CARDIO" class="0">
@@
 </segment>
 <segment>
-<pinref part="R6" gate="B" pin="2"/>
-<wire x1="337.82" y1="104.14" x2="335.28" y2="104.14" width="0.1524" layer="91"/>
-<label x="327.66" y="104.14" size="1.27" layer="95"/>
-</segment>
-</net>
+<pinref part="U1" gate="G$1" pin="PD16"/>
+<wire x1="215.9" y1="121.92" x2="220.98" y2="121.92" width="0.1524" layer="91"/>
+</segment>
+</net>

Commit message: tweak
Parts:
- C20, C21, C4: value 10u -> 4u7
Changed lines of the file:
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@@
 <part name="L4" library="jaw" deviceset="L" device="SMD0603" value="10uH"/>
 <part name="R2" library="jaw" deviceset="R" device="-0402" value="5k62 1%"/>
-<part name="C4" library="jaw" deviceset="C" device="0603" value="10u"/>
+<part name="C4" library="jaw" deviceset="C" device="0603" value="4u7"/>
 <part name="C5" library="jaw" deviceset="C" device="-0402" value="10p"/>
 <part name="GND3" library="jaw" deviceset="PWR-GND" device=""/>
@@
 <part name="SW1" library="jaw" deviceset="SWITCH" device="KMR211"/>
 <part name="SW2" library="jaw" deviceset="SWITCH" device="KMR211"/>
-<part name="C20" library="jaw" deviceset="C" device="0603" value="10u"/>
-<part name="C21" library="jaw" deviceset="C" device="0603" value="10u"/>
+<part name="C20" library="jaw" deviceset="C" device="0603" value="4u7"/>
+<part name="C21" library="jaw" deviceset="C" device="0603" value="4u7"/>
 <part name="C22" library="jaw" deviceset="C" device="0603" value="1u"/>
 <part name="C23" library="jaw" deviceset="C" device="-0402" value=".1u"/>
@@
 <pinref part="U1" gate="G$1" pin="PD16"/>
 <wire x1="215.9" y1="121.92" x2="220.98" y2="121.92" width="0.1524" layer="91"/>
-</segment>
-</net>
+<label x="220.98" y="121.92" size="1.27" layer="95"/>
+</segment>
+</net>

Commit message: move LEDs
Parts:
- added LED4: RED, jaw:LED
- LED2: value LED-DUAL0805 -> green; device jaw:LED-DUAL0805 -> jaw:LED
- LED3: value RED -> orange
Connections:
- net GND: now also LED2.C, LED3.C; no longer LED2.CB, LED2.CR
- net N$12: now also LED4.C; no longer LED3.C
- net N$4: now also LED2.A; no longer LED2.AB
- net N$5: now also LED3.A; no longer LED2.AR
- net PINA12: no longer U1.PA12
- net SWCLK: now also R4.P$1; no longer R12.P$1
- net SWDIO: now also R12.P$1; no longer R4.P$1
- net VIN: now also LED4.A; no longer LED3.A
Other:
- note added: "RX"
- note added: "TX"
- moved on the sheet: LED3, R12, R4
Changed lines of the file:
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@@
 <part name="R7" library="jaw" deviceset="R" device="-0402" value="1k"/>
 <part name="R8" library="jaw" deviceset="R" device="-0402" value="1k"/>
-<part name="LED2" library="jaw" deviceset="LED-DUAL" device="0805"/>
 <part name="Q1" library="jaw" deviceset="FDC6392S" device=""/>
 <part name="GND18" library="jaw" deviceset="PWR-GND" device=""/>
@@
 <part name="GND19" library="jaw" deviceset="PWR-GND" device=""/>
 <part name="GND20" library="jaw" deviceset="PWR-GND" device=""/>
-<part name="LED3" library="jaw" deviceset="LED" device="" value="RED"/>
+<part name="LED4" library="jaw" deviceset="LED" device="" value="RED"/>
 <part name="R11" library="jaw" deviceset="R" device="-0402" value="1k"/>
 <part name="CN6" library="jaw" deviceset="HEADER-1X1" device="SMALL" value="DO NOT PLACE"/>
 <part name="CN7" library="jaw" deviceset="HEADER-1X1" device="SMALL" value="DO NOT PLACE"/>
 <part name="C25" library="jaw" deviceset="C" device="0603" value="10u 10V"/>
+<part name="R12" library="jaw" deviceset="R" device="-0402" value="100k"/>
 <part name="R4" library="jaw" deviceset="R" device="-0402" value="100k"/>
-<part name="R12" library="jaw" deviceset="R" device="-0402" value="100k"/>
 <part name="VCC10" library="jaw" deviceset="PWR-VCC" device=""/>
+<part name="LED2" library="jaw" deviceset="LED" device="" value="green"/>
+<part name="LED3" library="jaw" deviceset="LED" device="" value="orange"/>
 </parts>
 <sheets>
@@
 does not include</text>
 <text x="73.66" y="50.8" size="1.27" layer="97">10k =&gt; 100mA charge</text>
+<text x="20.32" y="152.4" size="2.54" layer="97">RX</text>
+<text x="20.32" y="142.24" size="2.54" layer="97">TX</text>
 </plain>
 <instances>
@@
 <instance part="R7" gate="G$1" x="50.8" y="142.24"/>
 <instance part="R8" gate="G$1" x="50.8" y="152.4"/>
-<instance part="LED2" gate="G$1" x="40.64" y="147.32" rot="R180"/>
 <instance part="Q1" gate="G$1" x="91.44" y="60.96" rot="MR180"/>
 <instance part="GND18" gate="G$1" x="20.32" y="10.16"/>
@@
 <instance part="GND19" gate="G$1" x="68.58" y="45.72"/>
 <instance part="GND20" gate="G$1" x="106.68" y="68.58"/>
-<instance part="LED3" gate="G$1" x="17.78" y="55.88" rot="R270"/>
+<instance part="LED4" gate="G$1" x="17.78" y="55.88" rot="R270"/>
 <instance part="R11" gate="G$1" x="25.4" y="50.8" rot="R180"/>
 <instance part="CN6" gate="G$1" x="43.18" y="132.08"/>
 <instance part="CN7" gate="G$1" x="53.34" y="132.08" rot="R180"/>
 <instance part="C25" gate="G$1" x="40.64" y="15.24"/>
-<instance part="R4" gate="G$1" x="416.56" y="73.66" rot="R90"/>
-<instance part="R12" gate="G$1" x="421.64" y="73.66" rot="R90"/>
+<instance part="R12" gate="G$1" x="416.56" y="73.66" rot="R90"/>
+<instance part="R4" gate="G$1" x="421.64" y="73.66" rot="R90"/>
 <instance part="VCC10" gate="G$1" x="419.1" y="83.82"/>
+<instance part="LED2" gate="G$1" x="40.64" y="152.4" rot="R180"/>
+<instance part="LED3" gate="G$1" x="40.64" y="142.24" rot="R180"/>
 </instances>
 <busses>
@@
 <wire x1="35.56" y1="170.18" x2="30.48" y2="170.18" width="0.1524" layer="91"/>
 <wire x1="30.48" y1="170.18" x2="30.48" y2="152.4" width="0.1524" layer="91"/>
-<pinref part="LED2" gate="G$1" pin="CB"/>
 <wire x1="30.48" y1="152.4" x2="30.48" y2="142.24" width="0.1524" layer="91"/>
 <wire x1="30.48" y1="142.24" x2="30.48" y2="132.08" width="0.1524" layer="91"/>
@@
 <wire x1="35.56" y1="152.4" x2="30.48" y2="152.4" width="0.1524" layer="91"/>
 <junction x="30.48" y="152.4"/>
-<pinref part="LED2" gate="G$1" pin="CR"/>
 <wire x1="35.56" y1="142.24" x2="30.48" y2="142.24" width="0.1524" layer="91"/>
 <junction x="30.48" y="142.24"/>
@@
 <wire x1="35.56" y1="132.08" x2="30.48" y2="132.08" width="0.1524" layer="91"/>
 <junction x="30.48" y="132.08"/>
+<pinref part="LED2" gate="G$1" pin="C"/>
+<pinref part="LED3" gate="G$1" pin="C"/>
 </segment>
 <segment>
@@
 </segment>
 <segment>
+<pinref part="R12" gate="G$1" pin="P$2"/>
+<wire x1="416.56" y1="78.74" x2="416.56" y2="81.28" width="0.1524" layer="91"/>
 <pinref part="R4" gate="G$1" pin="P$2"/>
-<wire x1="416.56" y1="78.74" x2="416.56" y2="81.28" width="0.1524" layer="91"/>
-<pinref part="R12" gate="G$1" pin="P$2"/>
 <wire x1="416.56" y1="81.28" x2="419.1" y2="81.28" width="0.1524" layer="91"/>
 <wire x1="419.1" y1="81.28" x2="421.64" y2="81.28" width="0.1524" layer="91"/>
@@
 <wire x1="403.86" y1="63.5" x2="406.4" y2="63.5" width="0.1524" layer="91"/>
 <label x="406.4" y="63.5" size="1.27" layer="95"/>
-<pinref part="R12" gate="G$1" pin="P$1"/>
+<pinref part="R4" gate="G$1" pin="P$1"/>
 <wire x1="406.4" y1="63.5" x2="421.64" y2="63.5" width="0.1524" layer="91"/>
 <wire x1="421.64" y1="63.5" x2="421.64" y2="68.58" width="0.1524" layer="91"/>
@@
 <wire x1="403.86" y1="66.04" x2="406.4" y2="66.04" width="0.1524" layer="91"/>
 <label x="406.4" y="66.04" size="1.27" layer="95"/>
-<pinref part="R4" gate="G$1" pin="P$1"/>
+<pinref part="R12" gate="G$1" pin="P$1"/>
 <wire x1="406.4" y1="66.04" x2="416.56" y2="66.04" width="0.1524" layer="91"/>
 <wire x1="416.56" y1="66.04" x2="416.56" y2="68.58" width="0.1524" layer="91"/>
@@
 <wire x1="360.68" y1="193.04" x2="365.76" y2="193.04" width="0.1524" layer="91"/>
 <label x="365.76" y="193.04" size="1.27" layer="95"/>
-</segment>
-</net>
-<net name="N$4" class="0">
-<segment>
-<pinref part="LED2" gate="G$1" pin="AB"/>
-<pinref part="R8" gate="G$1" pin="P$1"/>
-</segment>
-</net>
-<net name="N$5" class="0">
-<segment>
-<pinref part="LED2" gate="G$1" pin="AR"/>
-<pinref part="R7" gate="G$1" pin="P$1"/>
 </segment>
 </net>
@@
 <pinref part="Q1" gate="G$1" pin="A"/>
 <pinref part="R10" gate="G$1" pin="P$2"/>
-<wire x1="96.52" y1="66.04" x2="96.52" y2="71.12" width="0.1524" layer="91"/>
-<junction x="96.52" y="66.04"/>
+<junction x="96.52" y="71.12"/>
 <wire x1="96.52" y1="71.12" x2="81.28" y2="71.12" width="0.1524" layer="91"/>
 <pinref part="Q1" gate="G$1" pin="G"/>
@@
 <pinref part="F1" gate="G$1" pin="2"/>
 <wire x1="30.48" y1="68.58" x2="30.48" y2="60.96" width="0.1524" layer="91"/>
-<wire x1="96.52" y1="66.04" x2="96.52" y2="71.12" width="0.1524" layer="91"/>
 <wire x1="81.28" y1="71.12" x2="30.48" y2="71.12" width="0.1524" layer="91"/>
 <wire x1="30.48" y1="71.12" x2="30.48" y2="68.58" width="0.1524" layer="91"/>
@@
 <wire x1="27.94" y1="71.12" x2="30.48" y2="71.12" width="0.1524" layer="91"/>
 <junction x="30.48" y="71.12"/>
-<pinref part="LED3" gate="G$1" pin="A"/>
+<pinref part="LED4" gate="G$1" pin="A"/>
 <wire x1="17.78" y1="60.96" x2="30.48" y2="60.96" width="0.1524" layer="91"/>
 <junction x="30.48" y="60.96"/>
+<wire x1="96.52" y1="71.12" x2="96.52" y2="66.04" width="0.1524" layer="91"/>
 </segment>
 </net>
@@
 <net name="PINA12" class="0">
 <segment>
-<pinref part="U1" gate="G$1" pin="PA12"/>
-<wire x1="170.18" y1="154.94" x2="165.1" y2="154.94" width="0.1524" layer="91"/>
-</segment>
-<segment>
 <pinref part="CN5" gate="A" pin="13"/>
 <wire x1="353.06" y1="203.2" x2="347.98" y2="203.2" width="0.1524" layer="91"/>
@@
 <segment>
 <pinref part="R11" gate="G$1" pin="P$2"/>
-<pinref part="LED3" gate="G$1" pin="C"/>
+<pinref part="LED4" gate="G$1" pin="C"/>
 <wire x1="20.32" y1="50.8" x2="17.78" y2="50.8" width="0.1524" layer="91"/>
 </segment>
 </net>
+<net name="N$4" class="0">
+<segment>
+<pinref part="R8" gate="G$1" pin="P$1"/>
+<pinref part="LED2" gate="G$1" pin="A"/>
+</segment>
+</net>
+<net name="N$5" class="0">
+<segment>
+<pinref part="R7" gate="G$1" pin="P$1"/>
+<pinref part="LED3" gate="G$1" pin="A"/>
+</segment>
+</net>

Commit message: piezo conn
Parts:
- removed CN6, CN7: DO NOT PLACE, jaw:HEADER-1X1SMALL
- added CN8: HEADER-1X2-THM, jaw:HEADER-1X2-THM
Connections:
- net GND: now also CN8.P$2; no longer CN6.P$1
- net PIEZO: now also CN8.P$1; no longer CN7.P$1
- net PINA12: now also U1.PA12
Changed lines of the file:
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@@
 <part name="LED4" library="jaw" deviceset="LED" device="" value="RED"/>
 <part name="R11" library="jaw" deviceset="R" device="-0402" value="1k"/>
-<part name="CN6" library="jaw" deviceset="HEADER-1X1" device="SMALL" value="DO NOT PLACE"/>
-<part name="CN7" library="jaw" deviceset="HEADER-1X1" device="SMALL" value="DO NOT PLACE"/>
 <part name="C25" library="jaw" deviceset="C" device="0603" value="10u 10V"/>
 <part name="R12" library="jaw" deviceset="R" device="-0402" value="100k"/>
@@
 <part name="LED2" library="jaw" deviceset="LED" device="" value="green"/>
 <part name="LED3" library="jaw" deviceset="LED" device="" value="orange"/>
+<part name="CN8" library="jaw" deviceset="HEADER-1X2" device="-THM"/>
 </parts>
 <sheets>
@@
 <instance part="LED4" gate="G$1" x="17.78" y="55.88" rot="R270"/>
 <instance part="R11" gate="G$1" x="25.4" y="50.8" rot="R180"/>
-<instance part="CN6" gate="G$1" x="43.18" y="132.08"/>
-<instance part="CN7" gate="G$1" x="53.34" y="132.08" rot="R180"/>
 <instance part="C25" gate="G$1" x="40.64" y="15.24"/>
 <instance part="R12" gate="G$1" x="416.56" y="73.66" rot="R90"/>
@@
 <instance part="LED2" gate="G$1" x="40.64" y="152.4" rot="R180"/>
 <instance part="LED3" gate="G$1" x="40.64" y="142.24" rot="R180"/>
+<instance part="CN8" gate="G$1" x="45.72" y="127" rot="R270"/>
 </instances>
 <busses>
@@
 <wire x1="35.56" y1="142.24" x2="30.48" y2="142.24" width="0.1524" layer="91"/>
 <junction x="30.48" y="142.24"/>
-<pinref part="CN6" gate="G$1" pin="P$1"/>
 <wire x1="35.56" y1="132.08" x2="30.48" y2="132.08" width="0.1524" layer="91"/>
 <junction x="30.48" y="132.08"/>
 <pinref part="LED2" gate="G$1" pin="C"/>
 <pinref part="LED3" gate="G$1" pin="C"/>
+<pinref part="CN8" gate="G$1" pin="P$2"/>
+<wire x1="45.72" y1="132.08" x2="35.56" y2="132.08" width="0.1524" layer="91"/>
 </segment>
 <segment>
@@
 </segment>
 <segment>
-<pinref part="CN7" gate="G$1" pin="P$1"/>
 <wire x1="60.96" y1="132.08" x2="63.5" y2="132.08" width="0.1524" layer="91"/>
 <label x="63.5" y="132.08" size="1.27" layer="95"/>
+<pinref part="CN8" gate="G$1" pin="P$1"/>
+<wire x1="48.26" y1="132.08" x2="60.96" y2="132.08" width="0.1524" layer="91"/>
 </segment>
 </net>
@@
 <label x="340.36" y="203.2" size="1.27" layer="95"/>
 </segment>
-</net>
+<segment>
+<pinref part="U1" gate="G$1" pin="PA12"/>
+<wire x1="170.18" y1="154.94" x2="165.1" y2="154.94" width="0.1524" layer="91"/>
+<label x="157.48" y="154.94" size="1.27" layer="95"/>
+</segment>
+</net>
