File: cad/se7en.sch (EAGLE design)
At the start: 67 parts, among them CN1 MICROSD-EJECT, CN3 DO NOT PLACE, CN4 DO NOT PLACE, CN5 DO NOT PLACE, CN8 DO NOT PLACE, Q1 FDC6392S, SW1 SWITCHKMR211, SW2 SWITCHKMR211, U1 ATSAMS70, U2 MCP73831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

Commit message: brighten green
Parts:
- R8: value 1k -> 470
Changed lines of the file:
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@@
 <part name="VR1" library="jaw" deviceset="REGULATOR4" device="-SOT23" value="3v3, 500mA"/>
 <part name="R7" library="jaw" deviceset="R" device="-0402" value="1k"/>
-<part name="R8" library="jaw" deviceset="R" device="-0402" value="1k"/>
+<part name="R8" library="jaw" deviceset="R" device="-0402" value="470"/>
 <part name="Q1" library="jaw" deviceset="FDC6392S" device=""/>
 <part name="GND18" library="jaw" deviceset="PWR-GND" device=""/>
